File: CUR_ground_station_25-26/Peripherals.kicad_sch (KiCad schematic)
At the start: 0 parts

Commit message: sgAdded usbc to peripherals page but actually this time
Parts:
- added J1: USB_C_Receptacle_USB2.0_16P, symbol Connector:USB_C_Receptacle_USB2.0_16P
- added R1, R2: R_US, symbol Device:R_US
- added U1: USBLC6-2SC6, Package_TO_SOT_SMD:SOT-23-6, symbol Power_Protection:USBLC6-2SC6
Connections:
- new net: J1.A5 (CC1), R1.1
- new net: J1.A7 (D-), J1.B7 (D-), U1.1 (I/O1)
- new net: J1.A6 (D+), J1.B6 (D+), U1.3 (I/O2)
- new net: J1.B5 (CC2), R2.1
- new net GND: J1.A1 (GND), J1.A12 (GND), J1.B1 (GND), J1.B12 (GND), J1.S1 (SHIELD), R1.2, R2.2, U1.2 (GND)
- new net USB_D+: U1.4 (I/O2)
- new net USB_D-: U1.6 (I/O1)
- new net VBUS: J1.A4 (VBUS), J1.A9 (VBUS), J1.B4 (VBUS), J1.B9 (VBUS), U1.5 (VBUS)
- no-connect marks 0 -> 2
Other:
- note added: "ESD Protection Place near connector"
