File: CUR_ground_station_25-26/Telemetry.kicad_sch (KiCad schematic)
At the start: 19 parts, among them J3 Conn_Coaxial_Small, U5 E22-400MM_22S

Commit message: Add MPNs
Parts:
- C6: MPN (none) -> CL10A105KO8NNNC
- J3: MPN (none) -> BWSMA-KE-P001
- R23: MPN (none) -> RC0603FR-0710KL
- R24, R25: MPN (none) -> RC0603FR-070RL
- U5: MPN (none) -> E22-400MM22S
Changed lines of the file:
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@@
+			)
+		)
+		(property "MPN" "RC0603FR-070RL"
+			(at 64.77 86.36 0)
+			(effects
+				(font
+					(size 1.27 1.27)
+				)
+				(hide yes)
 			)
 		)
@@
 			)
 		)
+		(property "MPN" "RC0603FR-070RL"
+			(at 110.49 60.96 90)
+			(effects
+				(font
+					(size 1.27 1.27)
+				)
+				(hide yes)
+			)
+		)
 		(pin "1"
 		)
@@
 			)
 		)
+		(property "MPN" "RC0603FR-0710KL"
+			(at 39.37 63.5 0)
+			(effects
+				(font
+					(size 1.27 1.27)
+				)
+				(hide yes)
+			)
+		)
 		(pin "1"
 		)
@@
 		)
 		(property "Description" "Unpolarized capacitor, small symbol"
+			(at 76.2 43.18 0)
+			(effects
+				(font
+					(size 1.27 1.27)
+				)
+				(hide yes)
+			)
+		)
+		(property "MPN" "CL10A105KO8NNNC"
 			(at 76.2 43.18 0)
 			(effects
@@
 			)
 		)
+		(property "MPN" "E22-400MM22S"
+			(at 83.82 58.42 0)
+			(effects
+				(font
+					(size 1.27 1.27)
+				)
+				(hide yes)
+			)
+		)
 		(pin "10"
 		)
@@
 			(at 128.27 60.96 0)
 			(effects
+				(font
+					(size 1.27 1.27)
+				)
+				(hide yes)
+			)
+		)
+		(property "MPN" "BWSMA-KE-P001"
+			(at 128.27 60.96 0)
+			(effects
